Commit message: add new world

File: description/lidar.xacro (robot description, xacro)
@@ -4,5 +4,5 @@
         <parent link="chassis_link"/>
         <child link="laser_frame"/>
-        <origin xyz="0.45 0 0.20" rpy="0 0 0"/>
+        <origin xyz="0.45 0 0.23" rpy="0 0 0"/>
     </joint>
     <link name="laser_frame">
@@ -18,5 +18,5 @@
             </geometry>
         </collision>
-        <xacro:inertial_cylinder mass="0.1" radius="0.05" length="0.04">
+        <xacro:inertial_cylinder mass="0.1" radius="0.05" length="0.08">
             <origin xyz="0 0 0" rpy="0 0 0"/>
         </xacro:inertial_cylinder>

File: description/robot.urdf.xacro (robot description, xacro)
@@ -4,3 +4,8 @@
     <xacro:include filename="gazebo_control.xacro"/>
     <xacro:include filename="lidar.xacro"/>
+    <xacro:include filename="gps.xacro"/>
+    <!-- <xacro:include filename="camera_front.xacro"/>
+    <xacro:include filename="camera_rear.xacro"/> -->
+    <xacro:include filename="depth_camera.xacro"/>
+    <xacro:include filename="imu.xacro"/>
 </robot>

File: description/robot_core.xacro (robot description, xacro)
@@ -40,5 +40,5 @@
             </geometry>
         </collision>
-        <xacro:inertial_box mass="3" x="0.6" y="0.6" z="0.2">
+        <xacro:inertial_box mass="5" x="0.6" y="0.6" z="0.2">
             <origin xyz="0.3 0 0.1" rpy="0 0 0"/>
         </xacro:inertial_box>
